File: Circuits/REFLECTEURS/REFLECTEURS.sch (KiCad schematic (older format))
At the start: 24 parts, among them P1 HE10-10, U1 3mm_hole, U2 3mm_hole

Commit message: Amelioration carte reflecteurs (simple face)
Parts:
- U1, U2: symbol 3mm_hole -> 3mm_hole-RESCUE-REFLECTEURS
Connections:
- net +1V5: now also P1.6; no longer P1.1
- net +5V: now also P1.4; no longer P1.2
- net GND: now also P1.8; no longer P1.10
- net at R2.1, REFL.1.2 (Coll): now also P1.10; no longer P1.4
- net at R4.1, REFL.2.2 (Coll): now also P1.9; no longer P1.6
- net at R6.1, REFL.3.2 (Coll): now also P1.7; no longer P1.8
- net at R8.1, REFL.4.2 (Coll): now also P1.5; no longer P1.9
- net at R10.1, REFL.5.2 (Coll): now also P1.3; no longer P1.7
- net at R12.1, REFL.6.2 (Coll): now also P1.1; no longer P1.5
- net at R14.1, REFL.7.2 (Coll): now also P1.2; no longer P1.3
Changed lines of the file:
@@
 EESchema Schematic File Version 2
+LIBS:REFLECTEURS-rescue
 LIBS:power
 LIBS:device
@@
 L +5V #PWR022
 U 1 1 575304F2
-P 5050 3200
-F 0 "#PWR022" H 5050 3050 50  0001 C CNN
-F 1 "+5V" H 5050 3340 50  0000 C CNN
-F 2 "" H 5050 3200 50  0000 C CNN
-F 3 "" H 5050 3200 50  0000 C CNN
-	1    5050 3200
+P 5050 3400
+F 0 "#PWR022" H 5050 3250 50  0001 C CNN
+F 1 "+5V" H 5050 3540 50  0000 C CNN
+F 2 "" H 5050 3400 50  0000 C CNN
+F 3 "" H 5050 3400 50  0000 C CNN
+	1    5050 3400
 	0    1    1    0
 $EndComp
@@
 L +1V5 #PWR023
 U 1 1 57530574
-P 3950 3200
-F 0 "#PWR023" H 3950 3050 50  0001 C CNN
-F 1 "+1V5" H 3950 3340 50  0000 C CNN
-F 2 "" H 3950 3200 50  0000 C CNN
-F 3 "" H 3950 3200 50  0000 C CNN
-	1    3950 3200
-	0    -1   -1   0
-$EndComp
-$Comp
-L 3mm_hole U1
+P 5050 3600
+F 0 "#PWR023" H 5050 3450 50  0001 C CNN
+F 1 "+1V5" H 5050 3740 50  0000 C CNN
+F 2 "" H 5050 3600 50  0000 C CNN
+F 3 "" H 5050 3600 50  0000 C CNN
+	1    5050 3600
+	0    1    1    0
+$EndComp
+$Comp
+L 3mm_hole-RESCUE-REFLECTEURS U1
 U 1 1 575339ED
 P 800 1300
@@
 $EndComp
 $Comp
-L 3mm_hole U2
+L 3mm_hole-RESCUE-REFLECTEURS U2
 U 1 1 57533B03
 P 5900 1300
@@
 	3500 1750 3700 1750
 Wire Wire Line
-	3700 1750 3700 2450
-Wire Wire Line
-	3700 2450 3150 2450
-Wire Wire Line
-	3150 2450 3150 4000
-Wire Wire Line
-	3150 4000 3950 4000
-Wire Wire Line
 	4200 1750 4400 1750
 Wire Wire Line
-	4400 1750 4400 2600
-Wire Wire Line
-	4400 2600 3250 2600
-Wire Wire Line
-	3250 2600 3250 3800
-Wire Wire Line
-	3250 3800 3950 3800
-Wire Wire Line
-	4850 1750 4950 1750
-Wire Wire Line
-	4950 1750 4950 2750
-Wire Wire Line
-	4950 2750 3400 2750
-Wire Wire Line
-	3400 2750 3400 3600
-Wire Wire Line
-	3400 3600 3950 3600
+	4850 1750 5000 1750
 Wire Wire Line
 	5500 1750 5750 1750
-Wire Wire Line
-	5750 1750 5750 2950
-Wire Wire Line
-	5750 2950 3550 2950
-Wire Wire Line
-	3550 2950 3550 3400
-Wire Wire Line
-	3550 3400 3950 3400
-Wire Wire Line
-	3000 1750 3000 4250
-Wire Wire Line
-	3000 4250 5300 4250
-Wire Wire Line
-	2400 1750 2400 4350
-Wire Wire Line
-	2400 4350 5350 4350
-Wire Wire Line
-	1700 1750 1700 4450
-Wire Wire Line
-	1700 4450 5400 4450
 $Comp
 L GND #PWR024
 U 1 1 57530486
-P 5050 4000
-F 0 "#PWR024" H 5050 3750 50  0001 C CNN
-F 1 "GND" H 5050 3850 50  0000 C CNN
-F 2 "" H 5050 4000 50  0000 C CNN
-F 3 "" H 5050 4000 50  0000 C CNN
-	1    5050 4000
+P 5050 3800
+F 0 "#PWR024" H 5050 3550 50  0001 C CNN
+F 1 "GND" H 5050 3650 50  0000 C CNN
+F 2 "" H 5050 3800 50  0000 C CNN
+F 3 "" H 5050 3800 50  0000 C CNN
+	1    5050 3800
 	0    -1   1    0
 $EndComp
 Wire Wire Line
-	5050 3800 5300 3800
-Wire Wire Line
-	5300 3800 5300 4250
-Wire Wire Line
-	5350 4350 5350 3600
-Wire Wire Line
-	5350 3600 5050 3600
-Wire Wire Line
-	5400 4450 5400 3400
-Wire Wire Line
-	5400 3400 5050 3400
+	1700 1750 1700 4300
+Wire Wire Line
+	1700 4300 5050 4300
+Wire Wire Line
+	5050 4300 5050 4000
+Wire Wire Line
+	3950 4000 2400 4000
+Wire Wire Line
+	2400 4000 2400 1750
+Wire Wire Line
+	3950 3800 3000 3800
+Wire Wire Line
+	3000 3800 3000 1750
+Wire Wire Line
+	3700 1750 3700 3600
+Wire Wire Line
+	3700 3600 3950 3600
+Wire Wire Line
+	3950 3400 3850 3400
+Wire Wire Line
+	3850 3400 3850 2300
+Wire Wire Line
+	3850 2300 4400 2300
+Wire Wire Line
+	4400 2300 4400 1750
+Wire Wire Line
+	3950 3200 3950 2450
+Wire Wire Line
+	3950 2450 5000 2450
+Wire Wire Line
+	5000 2450 5000 1750
+Wire Wire Line
+	5050 3200 5750 3200
+Wire Wire Line
+	5750 3200 5750 1750
 $EndSCHEMATC
